File: Switch de potencia.brd (EAGLE design)
At the start: 35 x 42 mm, 42 parts, among them U1 ATTINY828-AU32A_ATM-M, U3 AP63205WU-7SOIC_05WU-7_DIO-M

Commit message: Add files via upload
Parts:
- removed C1, C2: 22u, rcl:C0805
- removed C10, C9: (no value), rcl:C050-035X075
- removed POWERON1: (no value), led:CHIPLED_0603
- removed R10: (no value), rcl:M0805
- removed R9: 1.2k, rcl:M0805
- added POWERON4, POWERON5: (no value), led:CHIPLED_0603
- added R3, R4, R5, R6, R7: 1.2k, rcl:M0805
- added SW1: PTS647SK38SMTR2LFS, Push smd:PTS647SK38SMTR2LFS_CNK
- moved C6 65.0 mm to (18.2, 36.7)
- moved C8 54.6 mm to (18.2, 38.7)
- moved C13 43.3 mm to (20.4, 25.3), turned to 270 degrees
- moved C5 42.7 mm to (19.3, 15.9), turned to 90 degrees
- moved C11 41.6 mm to (23.1, 22.5)
- moved C12 40.5 mm to (19.2, 25.3), turned to 270 degrees
- moved TP9 38.9 mm to (22.4, 24.9)
- moved C3 38.3 mm to (27.6, 31.5)
- moved D11 33.2 mm to (26.9, 17.9), turned to 90 degrees
- moved C14 32.4 mm to (31.8, 23.6)
- moved D6 31.2 mm to (23.2, 19.5), turned to 180 degrees
- moved C4 27.9 mm to (27.1, 22.2), turned to 270 degrees
- moved POWERON3 26.9 mm to (28.8, 2.20), turned to 180 degrees
- moved POWERON2 25.4 mm to (26.9, 2.20), turned to 180 degrees
- moved D12 21.3 mm to (29.2, 17.4), turned to 270 degrees
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Connections:
- removed net N$35: POWERON1.A, R10.1
- removed net N$36: POWERON2.A, R9.2
- removed net N$37: R11.1, U1.26
- removed net N$38: POWERON3.A, R11.2
- new net N$10: R3.2, R4.1, U1.22
- new net N$11: POWERON5.A, U1.24
- new net N$12: POWERON3.A, U1.26
- new net N$13: POWERON4.A, U1.23
- new net N$14: POWERON2.C, POWERON3.C, POWERON4.C, POWERON5.C, R11.1
- new net N$17: R5.2, R6.1, R7.1, U1.20, U3.2
- new net N$18: R7.2, U1.17
- new net N$9: R5.1, SW1.1, SW1.2
- net +5V: no longer C1.1, C2.1, R10.2
- net GND: now also R11.2, R4.2, R6.2; no longer C1.2, C10.2, C2.2, C9.2, POWERON1.C, POWERON2.C, POWERON3.C
- net N$34: now also POWERON2.A; no longer R9.1
- net V+: now also R3.1, SW1.3, SW1.4; no longer C10.1, C9.1, U3.2
Routing:
- net GND: track 65.9 -> 140.4 mm, vias 0 -> 3
- net V+: track 6.93 -> 61.7 mm, vias 0 -> 3
- net +5V: track 0.00 -> 14.0 mm
- net N$6: track 0.00 -> 11.2 mm, vias 0 -> 2
- net N$4: track 0.00 -> 11.0 mm, vias 0 -> 2
- net N$3: track 0.00 -> 10.6 mm, vias 0 -> 2
- net N$5: track 0.00 -> 10.5 mm, vias 0 -> 2
- net N$14: track 0.00 -> 9.04 mm
- net N$17: track 0.00 -> 8.92 mm
- net N$9: track 0.00 -> 8.47 mm
- net N$15: track 0.00 -> 8.03 mm
- net N$12: track 0.00 -> 5.73 mm
- net N$13: track 0.00 -> 4.76 mm
- net N$34: track 0.00 -> 4.11 mm
- net N$11: track 0.00 -> 3.28 mm
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
Commit message: Add files via upload
Parts:
- removed TP2, TP3, TP4: TPB1,27, testpad:B1,27
- removed U1: ATTINY828-AU32A_ATM-M, nuevoattiny828:32A_ATM-M
- added U2: ATMEGA4808-AURTQFP32_PT_MCH-M, Atmega4808:TQFP32_PT_MCH-M
Connections:
- removed net N$12: POWERON3.A, U1.26
- removed net N$13: POWERON4.A, U1.23
- removed net N$34: POWERON2.A, U1.25
- new net AVDD: U2.18
- new net VDD: U2.28
- net +5V: no longer U1.18, U1.4
- net GND: no longer U1.21, U1.5
- net N$10: no longer U1.22
- net N$11: now also U2.2; no longer U1.24
- net N$17: now also U2.10; no longer U1.20
- net N$18: now also U2.5; no longer U1.17
- net N$20: now also U2.30; no longer U1.8
- net N$3: now also U2.27; no longer U1.27
- net N$4: now also POWERON3.A, U2.4; no longer TP2.TP, U1.28
- net N$5: now also POWERON2.A, U2.3; no longer TP3.TP, U1.29
- net N$6: now also POWERON4.A, U2.1; no longer TP4.TP, U1.30
Routing:
- net N$6: track 11.2 -> 0.00 mm, vias 2 -> 0
- net N$4: track 11.0 -> 0.00 mm, vias 2 -> 0
- net N$3: track 10.6 -> 0.00 mm, vias 2 -> 0
- net N$5: track 10.5 -> 0.00 mm, vias 2 -> 0
- net N$12: track 5.73 -> 0.00 mm
- net N$13: track 4.76 -> 0.00 mm
- net N$34: track 4.11 -> 0.00 mm
- net +5V: track 14.0 -> 11.5 mm
- net N$11: track 3.28 -> 2.15 mm

Commit message: Add files via upload
Parts:
- U2: value ATMEGA4808-AURTQFP32_PT_MCH-M -> ATMEGA4808-AURTQFP32_PT_MCH-L; device Atmega4808:TQFP32_PT_MCH-M -> Atmega4808:TQFP32_PT_MCH-L
- moved U2 31.3 mm to (23.3, 8.90), turned to 270 degrees
- moved R2 12.5 mm to (20.2, 18.9), turned to 270 degrees
- moved +15V 10.5 mm to (21.6, 19.0)
- moved C11 9.53 mm to (30.8, 16.9), turned to 90 degrees
- moved C5 8.98 mm to (28.1, 13.8), turned to 180 degrees
- moved C4 4.68 mm to (31.6, 20.7), turned to 180 degrees
- moved R4 4.06 mm to (30.5, 9.10)
- moved D12 3.94 mm to (25.6, 19.0), turned to 90 degrees
- moved R3 2.82 mm to (31.5, 12.2)
- moved D2 2.00 mm to (22.1, 15.1), turned to 180 degrees
- moved D11 1.63 mm to (28.1, 19.0)
- moved C14 0.68 mm to (31.6, 22.9), turned to 180 degrees
- moved D6 0.53 mm to (23.2, 19.0), turned to 270 degrees
- moved PADGND 0.41 mm to (19.4, 22.9)
Connections:
- removed net AVDD: U2.18
- removed net VDD: U2.28
- net +5V: now also U2.18, U2.28
- net GND: now also U2.19, U2.29
- net N$10: now also U2.11
- net N$11: now also POWERON4.A, U2.21; no longer POWERON5.A, U2.2
- net N$18: now also U2.9; no longer U2.5
- net N$4: now also U2.24; no longer U2.4
- net N$5: now also U2.23; no longer U2.3
- net N$6: now also POWERON5.A, U2.22; no longer POWERON4.A, U2.1
Routing:
- net N$18: track 0.00 -> 49.6 mm, vias 0 -> 2
- net +5V: track 11.5 -> 40.7 mm
- net N$17: track 8.92 -> 32.2 mm, vias 0 -> 2
- net GND: track 140.4 -> 161.7 mm, vias 3 -> 6
- net N$7: track 0.00 -> 18.4 mm
- net N$10: track 0.00 -> 16.3 mm, vias 0 -> 4
- net V+: track 61.7 -> 76.2 mm, vias 3 -> 4
- net N$40: track 0.00 -> 10.1 mm, vias 0 -> 2
- net N$39: track 0.00 -> 8.36 mm
- net N$20: track 0.00 -> 7.85 mm
- net N$3: track 0.00 -> 6.45 mm
- net N$8: track 0.00 -> 6.30 mm
- net N$4: track 0.00 -> 4.04 mm
- net N$1: track 30.6 -> 33.8 mm, vias 3 -> 4
- net N$5: track 0.00 -> 3.12 mm
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- added copper zone on layer 1, net +5V
- added copper zone on layer 1, net GND
- added copper zone on layer 16, net GND
- added copper zone on layer 1, net N$2
Other:
- board text added: "Diseñado en México por Sol"
