File: Switch de potencia.brd (EAGLE design)
At the start: 35 x 42 mm, 40 parts, among them SW1 PTS647SK38SMTR2LFS, U2 ATMEGA4808-AURTQFP32_PT_MCH-L, U3 AP63205WU-7SOIC_05WU-7_DIO-M

Commit message: Add files via upload
Parts:
- removed SW1: PTS647SK38SMTR2LFS, Push smd:PTS647SK38SMTR2LFS_CNK
- added X1: 22-23-2021, con-molex:22-23-2021
Connections:
- net N$9: now also X1.2; no longer SW1.1, SW1.2
- net V+: now also X1.1; no longer SW1.3, SW1.4
Routing:
- net V+: track 76.2 -> 70.6 mm
- net N$9: track 8.47 -> 5.83 mm
Changed lines of the file:
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@@
 <attribute name="NAME" x="17.69" y="33.47" size="1.27" layer="25" rot="R180"/>
-</element>
-<element name="SW1" library="Push smd" package="PTS647SK38SMTR2LFS_CNK" value="PTS647SK38SMTR2LFS" x="29.1" y="38.2" smashed="yes" rot="R180">
-<attribute name="BUILT_BY" value="EMA_Cory" x="29.1" y="38.2" size="1.778" layer="27" rot="R180" display="off"/>
-<attribute name="COPYRIGHT" value="Copyright (C) 2018 Accelerated Designs. All rights reserved" x="29.1" y="38.2" size="1.778" layer="27" rot="R180" display="off"/>
-<attribute name="DATASHEET" value="https://www.ckswitches.com/media/2567/pts647.pdf" x="29.1" y="38.2" size="1.778" layer="27" rot="R180" display="off"/>
-<attribute name="MANUFACTURER_PART_NUMBER" value="PTS647SK38SMTR2LFS" x="29.1" y="38.2" size="1.778" layer="27" rot="R180" display="off"/>
-<attribute name="SOURCELIBRARY" value="C&amp;K_2020-05-06" x="29.1" y="38.2" size="1.778" layer="27" rot="R180" display="off"/>
-<attribute name="VENDOR" value="C&amp;K" x="29.1" y="38.2" size="1.778" layer="27" rot="R180" display="off"/>
 </element>
 <element name="R3" library="rcl" library_urn="urn:adsk.eagle:library:334" package="M0805" package3d_urn="urn:adsk.eagle:package:23556/2" value="1.2k" x="31.5" y="12.2" smashed="yes" rot="R270">
@@
 <attribute name="SOURCELIBRARY" value="Add_to_database_2021-02-15" x="23.3" y="8.9" size="1.778" layer="27" rot="R270" display="off"/>
 <attribute name="VENDOR" value="Microchip" x="23.3" y="8.9" size="1.778" layer="27" rot="R270" display="off"/>
+</element>
+<element name="X1" library="con-molex" library_urn="urn:adsk.eagle:library:165" package="22-23-2021" package3d_urn="urn:adsk.eagle:package:8078633/1" value="22-23-2021" x="29.4" y="37.5" smashed="yes">
+<attribute name="MF" value="MOLEX" x="29.4" y="37.5" size="1.778" layer="27" display="off"/>
+<attribute name="MPN" value="22-23-2021" x="29.4" y="37.5" size="1.778" layer="27" display="off"/>
+<attribute name="NAME" x="26.86" y="41.31" size="1.016" layer="25" ratio="10"/>
+<attribute name="OC_FARNELL" value="1462926" x="29.4" y="37.5" size="1.778" layer="27" display="off"/>
+<attribute name="OC_NEWARK" value="25C3832" x="29.4" y="37.5" size="1.778" layer="27" display="off"/>
+<attribute name="POPULARITY" value="40" x="29.4" y="37.5" size="1.778" layer="27" display="off"/>
+<attribute name="VALUE" x="26.86" y="32.42" size="1.016" layer="27" ratio="10"/>
 </element>
 </elements>
@@
 <wire x1="14.42" y1="37.74" x2="12.3" y2="37.74" width="2.54" layer="1"/>
 <contactref element="R3" pad="1"/>
-<contactref element="SW1" pad="3"/>
-<contactref element="SW1" pad="4"/>
 <wire x1="12.3" y1="37.74" x2="8.39" y2="37.74" width="2.54" layer="1"/>
 <wire x1="8.39" y1="37.74" x2="8" y2="37.64" width="2.54" layer="1"/>
-<wire x1="31.725" y1="39.8" x2="29.2" y2="39.8" width="1.016" layer="1"/>
-<wire x1="29.2" y1="39.8" x2="26.475" y2="39.8" width="1.016" layer="1"/>
-<wire x1="29.2" y1="39.8" x2="24.7" y2="39.8" width="0.508" layer="1"/>
-<wire x1="24.7" y1="39.8" x2="24.4" y2="39.5" width="0.508" layer="1"/>
 <via x="24.4" y="39.5" extent="1-16" drill="0.35"/>
 <wire x1="24.4" y1="39.5" x2="20.4" y2="35.5" width="0.508" layer="16"/>
@@
 <wire x1="33" y1="14.6" x2="33" y2="21.6" width="0.508" layer="16"/>
 <wire x1="33" y1="21.6" x2="29.2" y2="25.4" width="0.508" layer="16"/>
+<contactref element="X1" pad="1"/>
+<wire x1="24.4" y1="39.5" x2="26.13" y2="39.5" width="0.508" layer="1"/>
+<wire x1="26.13" y1="39.5" x2="28.13" y2="37.5" width="0.508" layer="1"/>
 </signal>
 <signal name="N$9">
-<contactref element="SW1" pad="1"/>
-<contactref element="SW1" pad="2"/>
 <contactref element="R5" pad="1"/>
-<wire x1="31.725" y1="36.6" x2="26.475" y2="36.6" width="1.016" layer="1"/>
-<wire x1="31.725" y1="36.6" x2="33.1" y2="35.225" width="1.016" layer="1"/>
 <wire x1="33.1" y1="35.225" x2="33.1" y2="33.95" width="1.016" layer="1"/>
+<contactref element="X1" pad="2"/>
+<wire x1="30.67" y1="37.5" x2="33.1" y2="35.07" width="0.508" layer="1"/>
+<wire x1="33.1" y1="35.07" x2="33.1" y2="33.95" width="0.508" layer="1"/>
 </signal>
 <signal name="N$10">

Commit message: Add files via upload
Agregue usart , un pin para recibir datos
Parts:
- added SV1: (no value), con-lstb:MA03-1
- moved R11 4.70 mm to (27.5, 1.97)
- moved POWERON3 4.10 mm to (24.7, 2.30)
- moved TP1 3.44 mm to (29.4, 5.93)
- moved POWERON2 3.40 mm to (23.6, 2.30)
- moved POWERON5 2.50 mm to (22.3, 2.30)
- moved POWERON4 1.40 mm to (21.0, 2.30)
Connections:
- new net N$12: SV1.3, U2.31
- net +5V: now also SV1.2
- net GND: now also SV1.1
- net N$11: now also U2.17; no longer U2.21
Routing:
- net N$12: track 0.00 -> 10.4 mm, vias 0 -> 1
- net +5V: track 40.7 -> 50.1 mm
- net V+: track 70.6 -> 65.0 mm
- net N$14: track 9.04 -> 5.74 mm
- net N$3: track 6.45 -> 3.77 mm
- net N$4: track 4.04 -> 2.12 mm
- net N$6: track 2.09 -> 3.03 mm
- net N$10: track 16.3 -> 17.0 mm
- net N$11: track 2.38 -> 1.78 mm
- net N$5: track 3.12 -> 2.58 mm
