File: Switch de potencia.sch (EAGLE design)
At the start: 42 parts, among them U1 ATTINY828-AU32A_ATM-M, U3 AP63205WU-7SOIC_05WU-7_DIO-M

Commit message: Add files via upload
Parts:
- removed C1, C2: 22u, rcl:C-EUC0805
- removed C10, C9: (no value), rcl:C-EU050-035X075
- removed POWERON1: (no value), led:LEDCHIPLED_0603
- removed R10: (no value), rcl:R-EU_M0805
- removed R9: 1.2k, rcl:R-EU_M0805
- added POWERON4, POWERON5: (no value), led:LEDCHIPLED_0603
- added R3, R4, R5, R6, R7: 1.2k, rcl:R-EU_M0805
- added SW1: PTS647SK38SMTR2LFS, Push smd:PTS647SK38SMTR2LFS
Connections:
- removed net N$35: POWERON1.A, R10.1
- removed net N$36: POWERON2.A, R9.2
- removed net N$37: R11.1, U1A.PB7
- removed net N$38: POWERON3.A, R11.2
- new net N$10: R3.2, R4.1, U1A.PB3
- new net N$11: POWERON5.A, U1A.PB5
- new net N$12: POWERON3.A, U1A.PB7
- new net N$13: POWERON4.A, U1A.PB4
- new net N$14: POWERON2.C, POWERON3.C, POWERON4.C, POWERON5.C, R11.1
- new net N$17: R5.2, R6.1, R7.1, U1A.PB2, U3.EN
- new net N$18: R7.2, U1A.PB0
- new net N$9: R5.1, SW1.1, SW1.2
- net +5V: no longer C1.1, C2.1, R10.2
- net GND: now also R11.2, R4.2, R6.2; no longer C1.2, C10.2, C2.2, C9.2, POWERON1.C, POWERON2.C, POWERON3.C
- net N$34: now also POWERON2.A; no longer R9.1
- net V+: now also R3.1, SW1.3, SW1.4; no longer C10.1, C9.1, U3.EN
Other:
- moved on the sheet: C3, C6, R11

Commit message: Add files via upload
Parts:
- removed TP2, TP3, TP4: TPB1,27, testpad:TPB1,27
- removed U1: ATTINY828-AU32A_ATM-M, nuevoattiny828:ATTINY828-AU32A_ATM-M
- added U2: ATMEGA4808-AURTQFP32_PT_MCH-M, Atmega4808:ATMEGA4808-AURTQFP32_PT_MCH-M
Connections:
- removed net N$12: POWERON3.A, U1A.PB7
- removed net N$13: POWERON4.A, U1A.PB4
- removed net N$34: POWERON2.A, U1A.PB6
- net +5V: no longer U1B.AVCC, U1B.VCC
- net GND: no longer U1B.GND, U1B.GND_2
- net N$10: no longer U1A.PB3
- net N$11: now also U2.PA4; no longer U1A.PB5
- net N$17: now also U2.PD0; no longer U1A.PB2
- net N$18: now also U2.PA7; no longer U1A.PB0
- net N$20: now also U2.PA0(EXTCLK); no longer U1A.PC7
- net N$3: now also U2.UPDI; no longer U1A.PD0
- net N$4: now also POWERON3.A, U2.PA6; no longer TP2.TP, U1A.PD1
- net N$5: now also POWERON2.A, U2.PA5; no longer TP3.TP, U1A.PD2
- net N$6: now also POWERON4.A, U2.PA3; no longer TP4.TP, U1A.PD3

Commit message: Add files via upload
Parts:
- U2: value ATMEGA4808-AURTQFP32_PT_MCH-M -> ATMEGA4808-AURTQFP32_PT_MCH-L; device Atmega4808:ATMEGA4808-AURTQFP32_PT_MCH-M -> Atmega4808:ATMEGA4808-AURTQFP32_PT_MCH-L
Connections:
- net +5V: now also U2.AVDD, U2.VDD
- net GND: now also U2.GND, U2.GND_2
- net N$10: now also U2.PD1
- net N$11: now also POWERON4.A, U2.PF1(TOSC2); no longer POWERON5.A, U2.PA4
- net N$18: now also U2.PC3; no longer U2.PA7
- net N$4: now also U2.PF4; no longer U2.PA6
- net N$5: now also U2.PF3; no longer U2.PA5
- net N$6: now also POWERON5.A, U2.PF2; no longer POWERON4.A, U2.PA3
Other:
- moved on the sheet: R1, R11, R4

Commit message: Add files via upload
Parts:
- removed SW1: PTS647SK38SMTR2LFS, Push smd:PTS647SK38SMTR2LFS
- added X1: 22-23-2021, con-molex:22-23-2021
Connections:
- net N$9: now also X1-2.S; no longer SW1.1, SW1.2
- net V+: now also X1-1.S; no longer SW1.3, SW1.4

Commit message: Add files via upload
Agregue usart , un pin para recibir datos
Parts:
- added SV1: (no value), con-lstb:MA03-1
Connections:
- new net N$12: SV1.3, U2.PA1
- net +5V: now also SV1.2
- net GND: now also SV1.1
- net N$11: now also U2.PD7; no longer U2.PF1(TOSC2)
Changed lines of the file:
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@@
 <part name="P+3" library="supply1" library_urn="urn:adsk.eagle:library:371" deviceset="+5V" device=""/>
 <part name="X1" library="con-molex" library_urn="urn:adsk.eagle:library:165" deviceset="22-23-2021" device="" package3d_urn="urn:adsk.eagle:package:8078633/1"/>
+<part name="SV1" library="con-lstb" library_urn="urn:adsk.eagle:library:162" deviceset="MA03-1" device="" package3d_urn="urn:adsk.eagle:package:8339/1"/>
 </parts>
 <sheets>
@@
 <instance part="X1" gate="-2" x="-160.02" y="71.12" smashed="yes" rot="R180">
 <attribute name="NAME" x="-162.56" y="71.882" size="1.524" layer="95" rot="R180"/>
+</instance>
+<instance part="SV1" gate="G$1" x="33.02" y="50.8" smashed="yes" rot="R180">
+<attribute name="VALUE" x="34.29" y="58.42" size="1.778" layer="96" rot="R180"/>
+<attribute name="NAME" x="34.29" y="44.958" size="1.778" layer="95" rot="R180"/>
 </instance>
 </instances>
@@
 <wire x1="5.08" y1="40.64" x2="20.32" y2="40.64" width="0.1524" layer="91"/>
 <wire x1="20.32" y1="40.64" x2="20.32" y2="35.56" width="0.1524" layer="91"/>
+<pinref part="SV1" gate="G$1" pin="1"/>
+<wire x1="25.4" y1="53.34" x2="20.32" y2="53.34" width="0.1524" layer="91"/>
+<wire x1="20.32" y1="53.34" x2="20.32" y2="40.64" width="0.1524" layer="91"/>
+<junction x="20.32" y="40.64"/>
 </segment>
 </net>
@@
 <wire x1="15.24" y1="33.02" x2="15.24" y2="38.1" width="0.1524" layer="91"/>
 <junction x="15.24" y="38.1"/>
+<pinref part="SV1" gate="G$1" pin="2"/>
+<wire x1="25.4" y1="50.8" x2="22.86" y2="50.8" width="0.1524" layer="91"/>
+<wire x1="22.86" y1="50.8" x2="22.86" y2="38.1" width="0.1524" layer="91"/>
+<wire x1="22.86" y1="38.1" x2="15.24" y2="38.1" width="0.1524" layer="91"/>
 </segment>
 </net>
@@
 </segment>
 </net>
+<net name="N$12" class="0">
+<segment>
+<pinref part="U2" gate="A" pin="PA1"/>
+<wire x1="5.08" y1="45.72" x2="10.16" y2="45.72" width="0.1524" layer="91"/>
+<wire x1="10.16" y1="45.72" x2="10.16" y2="48.26" width="0.1524" layer="91"/>
+<pinref part="SV1" gate="G$1" pin="3"/>
+<wire x1="10.16" y1="48.26" x2="25.4" y2="48.26" width="0.1524" layer="91"/>
+</segment>
+</net>
 <net name="N$11" class="0">
 <segment>
+<pinref part="U2" gate="A" pin="PD7"/>
+<wire x1="5.08" y1="10.16" x2="10.16" y2="10.16" width="0.1524" layer="91"/>
+<wire x1="10.16" y1="10.16" x2="10.16" y2="-2.54" width="0.1524" layer="91"/>
 <pinref part="POWERON4" gate="G$1" pin="A"/>
-<wire x1="24.13" y1="15.24" x2="17.78" y2="15.24" width="0.1524" layer="91"/>
-<wire x1="17.78" y1="15.24" x2="17.78" y2="20.32" width="0.1524" layer="91"/>
-<pinref part="U2" gate="A" pin="PF1(TOSC2)"/>
-<wire x1="17.78" y1="20.32" x2="5.08" y2="20.32" width="0.1524" layer="91"/>
-</segment>
-</net>
+<wire x1="10.16" y1="-2.54" x2="24.13" y2="-2.54" width="0.1524" layer="91"/>
+<wire x1="24.13" y1="-2.54" x2="24.13" y2="15.24" width="0.1524" layer="91"/>
+</segment>
+</net>
